File: MainPCB/Env-KB60F.kicad_pcb (KiCad board)
At the start: 2 copper layers, 283 x 126.5 mm, 149 parts, among them J1 TP3 Pad, J2 TP2 Pad, SW1 EVQ-P7A01P, U1 Pico

Commit message: Corrected mount hole placement on all PCBs and updated the switch plate to fit triple spacebar split.
Parts:
- moved H1 5.00 mm to (227.5, 155.0)
- renumbered D_59M to D_59, D_59L to D_590, D_59R to D_591
Connections:
- H1 pad 1: (no net) -> GND
- H10 pad 1: (no net) -> GND
- H11 pad 1: (no net) -> GND
- H2 pad 1: (no net) -> GND
- H3 pad 1: (no net) -> GND
- H4 pad 1: (no net) -> GND
- H6 pad 1: (no net) -> GND
- H9 pad 1: (no net) -> GND
