File: MainPCB/Env-KB60F.sch (KiCad schematic (older format))
At the start: 145 parts, among them J1 TP3 Pad, J2 TP2 Pad, SW1 EVQ-P7A01P, U1 Pico

Commit message: Moved MCU lower to allow for mount hole to fit properly, Generated Gerber and bottom plate Gerber
Parts:
- SW1: symbol PanasonicEVQ-P7A01P:EVQ-P7A01P -> Env-KB60F-rescue:EVQ-P7A01P-PanasonicEVQ-P7A01P
Changed lines of the file:
@@
 GND
 $Comp
-L PanasonicEVQ-P7A01P:EVQ-P7A01P SW1
+L Env-KB60F-rescue:EVQ-P7A01P-PanasonicEVQ-P7A01P SW1
 U 1 1 6096F576
 P 3900 5950

Commit message: Corrected silkscreen, Generated updated Gerbers
Parts:
- SW1: automotive No -> (none); category Switch -> (none); contact current rating 50mA -> (none); contact resistance 500mΩ -> (none); device class L1 Electromechanical -> (none); device class L2 Switches -> (none); device class L3 Tactile Switches -> (none); digikey description SWITCH TACTILE SPST-NO 0.05A 12V -> (none); digikey part number P16763CT-ND -> (none); electromechanical life 100000Cycles -> (none); height 1.55mm -> (none); lead free Yes -> (none); library id 2f293019bba4f771 -> (none); manufacturer Panasonic -> (none); mount Surface Mount -> (none); mouser description SWITCH TACTILE SPST-NO 0.05A 12V -> (none); mouser part number 667-EVQP7A01P -> (none); operating force 2.2N -> (none); package SMT_SW_3MM5_2MM9 -> (none); rohs Yes -> (none); temperature range high +70°C -> (none); temperature range low -20°C -> (none); throw configuration SPST-NO -> (none); voltage rating DC 12V -> (none)
Changed lines of the file:
@@
 F 2 "PanasonicEVQ-P7A01P:Panasonic-EVQ-P7A01P-0-0-MFG" H 3900 6150 50  0001 L CNN
 F 3 "https://industrial.panasonic.com/cdbs/www-data/pdf/ATK0000/ATK0000C378.pdf" H 3900 6250 50  0001 L CNN
-F 4 "No" H 3900 6350 50  0001 L CNN "automotive"
-F 5 "Switch" H 3900 6450 50  0001 L CNN "category"
-F 6 "50mA" H 3900 6550 50  0001 L CNN "contact current rating"
-F 7 "500mΩ" H 3900 6650 50  0001 L CNN "contact resistance"
-F 8 "Electromechanical" H 3900 6750 50  0001 L CNN "device class L1"
-F 9 "Switches" H 3900 6850 50  0001 L CNN "device class L2"
-F 10 "Tactile Switches" H 3900 6950 50  0001 L CNN "device class L3"
-F 11 "SWITCH TACTILE SPST-NO 0.05A 12V" H 3900 7050 50  0001 L CNN "digikey description"
-F 12 "P16763CT-ND" H 3900 7150 50  0001 L CNN "digikey part number"
-F 13 "100000Cycles" H 3900 7250 50  0001 L CNN "electromechanical life"
-F 14 "1.55mm" H 3900 7350 50  0001 L CNN "height"
-F 15 "Yes" H 3900 7450 50  0001 L CNN "lead free"
-F 16 "2f293019bba4f771" H 3900 7550 50  0001 L CNN "library id"
-F 17 "Panasonic" H 3900 7650 50  0001 L CNN "manufacturer"
-F 18 "Surface Mount" H 3900 7750 50  0001 L CNN "mount"
-F 19 "SWITCH TACTILE SPST-NO 0.05A 12V" H 3900 7850 50  0001 L CNN "mouser description"
-F 20 "667-EVQP7A01P" H 3900 7950 50  0001 L CNN "mouser part number"
-F 21 "2.2N" H 3900 8050 50  0001 L CNN "operating force"
-F 22 "SMT_SW_3MM5_2MM9" H 3900 8150 50  0001 L CNN "package"
-F 23 "Yes" H 3900 8250 50  0001 L CNN "rohs"
-F 24 "+70°C" H 3900 8350 50  0001 L CNN "temperature range high"
-F 25 "-20°C" H 3900 8450 50  0001 L CNN "temperature range low"
-F 26 "SPST-NO" H 3900 8550 50  0001 L CNN "throw configuration"
-F 27 "12V" H 3900 8650 50  0001 L CNN "voltage rating DC"
 	1    3900 5950
 	-1   0    0    1

Commit message: General Checkover and adjustments, Generated Gerbers for JLCPCB
Parts:
- 5.1K1, 5.1K2: value R_Small -> 5.1K 0402 Resistor; footprint Resistor_SMD:R_0201_0603Metric -> Resistor_SMD:R_0402_1005Metric
Changed lines of the file:
@@
 P 1900 7250
 F 0 "5.1K2" V 1900 7250 20  0000 C CNN
-F 1 "R_Small" V 1850 7250 20  0000 C CNN
-F 2 "Resistor_SMD:R_0201_0603Metric" H 1900 7250 50  0001 C CNN
+F 1 "5.1K 0402 Resistor" V 1850 7250 20  0000 C CNN
+F 2 "Resistor_SMD:R_0402_1005Metric" H 1900 7250 50  0001 C CNN
 F 3 "~" H 1900 7250 50  0001 C CNN
 	1    1900 7250
@@
 P 1900 6650
 F 0 "5.1K1" V 1900 6650 20  0000 C CNN
-F 1 "R_Small" V 1950 6650 20  0000 C CNN
-F 2 "Resistor_SMD:R_0201_0603Metric" H 1900 6650 50  0001 C CNN
+F 1 "5.1K 0402 Resistor" V 1950 6650 20  0000 C CNN
+F 2 "Resistor_SMD:R_0402_1005Metric" H 1900 6650 50  0001 C CNN
 F 3 "~" H 1900 6650 50  0001 C CNN
 	1    1900 6650

Commit message: Generated DXF for CNC or Laser cut.
Parts:
- H1, H10, H11, H2, H3, H4, H5, H6, H7, H9: footprint MountingHole:MountingHole_2.2mm_M2 -> AKLogo:MountingHole_2.2mm_M2-MODIFIED
Changed lines of the file:
@@
 F 0 "H1" H 5700 6396 50  0000 L CNN
 F 1 "MountingHole" H 5700 6305 50  0000 L CNN
-F 2 "MountingHole:MountingHole_2.2mm_M2" H 5600 6350 50  0001 C CNN
+F 2 "AKLogo:MountingHole_2.2mm_M2-MODIFIED" H 5600 6350 50  0001 C CNN
 F 3 "~" H 5600 6350 50  0001 C CNN
 	1    5600 6350
@@
 F 0 "H3" H 5700 6596 50  0000 L CNN
 F 1 "MountingHole" H 5700 6505 50  0000 L CNN
-F 2 "MountingHole:MountingHole_2.2mm_M2" H 5600 6550 50  0001 C CNN
+F 2 "AKLogo:MountingHole_2.2mm_M2-MODIFIED" H 5600 6550 50  0001 C CNN
 F 3 "~" H 5600 6550 50  0001 C CNN
 	1    5600 6550
@@
 F 0 "H5" H 5700 6796 50  0000 L CNN
 F 1 "MountingHole" H 5700 6705 50  0000 L CNN
-F 2 "MountingHole:MountingHole_2.2mm_M2" H 5600 6750 50  0001 C CNN
+F 2 "AKLogo:MountingHole_2.2mm_M2-MODIFIED" H 5600 6750 50  0001 C CNN
 F 3 "~" H 5600 6750 50  0001 C CNN
 	1    5600 6750
@@
 F 0 "H7" H 5700 6996 50  0000 L CNN
 F 1 "MountingHole" H 5700 6905 50  0000 L CNN
-F 2 "MountingHole:MountingHole_2.2mm_M2" H 5600 6950 50  0001 C CNN
+F 2 "AKLogo:MountingHole_2.2mm_M2-MODIFIED" H 5600 6950 50  0001 C CNN
 F 3 "~" H 5600 6950 50  0001 C CNN
 	1    5600 6950
@@
 F 0 "H9" H 5700 7196 50  0000 L CNN
 F 1 "MountingHole" H 5700 7105 50  0000 L CNN
-F 2 "MountingHole:MountingHole_2.2mm_M2" H 5600 7150 50  0001 C CNN
+F 2 "AKLogo:MountingHole_2.2mm_M2-MODIFIED" H 5600 7150 50  0001 C CNN
 F 3 "~" H 5600 7150 50  0001 C CNN
 	1    5600 7150
@@
 F 0 "H10" H 5700 7396 50  0000 L CNN
 F 1 "MountingHole" H 5700 7305 50  0000 L CNN
-F 2 "MountingHole:MountingHole_2.2mm_M2" H 5600 7350 50  0001 C CNN
+F 2 "AKLogo:MountingHole_2.2mm_M2-MODIFIED" H 5600 7350 50  0001 C CNN
 F 3 "~" H 5600 7350 50  0001 C CNN
 	1    5600 7350
@@
 F 0 "H11" H 5700 7596 50  0000 L CNN
 F 1 "MountingHole" H 5700 7505 50  0000 L CNN
-F 2 "MountingHole:MountingHole_2.2mm_M2" H 5600 7550 50  0001 C CNN
+F 2 "AKLogo:MountingHole_2.2mm_M2-MODIFIED" H 5600 7550 50  0001 C CNN
 F 3 "~" H 5600 7550 50  0001 C CNN
 	1    5600 7550
@@
 F 0 "H2" H 6500 6396 50  0000 L CNN
 F 1 "MountingHole" H 6500 6305 50  0000 L CNN
-F 2 "MountingHole:MountingHole_2.2mm_M2" H 6400 6350 50  0001 C CNN
+F 2 "AKLogo:MountingHole_2.2mm_M2-MODIFIED" H 6400 6350 50  0001 C CNN
 F 3 "~" H 6400 6350 50  0001 C CNN
 	1    6400 6350
@@
 F 0 "H4" H 6500 6596 50  0000 L CNN
 F 1 "MountingHole" H 6500 6505 50  0000 L CNN
-F 2 "MountingHole:MountingHole_2.2mm_M2" H 6400 6550 50  0001 C CNN
+F 2 "AKLogo:MountingHole_2.2mm_M2-MODIFIED" H 6400 6550 50  0001 C CNN
 F 3 "~" H 6400 6550 50  0001 C CNN
 	1    6400 6550
@@
 F 0 "H6" H 6500 6796 50  0000 L CNN
 F 1 "MountingHole" H 6500 6705 50  0000 L CNN
-F 2 "MountingHole:MountingHole_2.2mm_M2" H 6400 6750 50  0001 C CNN
+F 2 "AKLogo:MountingHole_2.2mm_M2-MODIFIED" H 6400 6750 50  0001 C CNN
 F 3 "~" H 6400 6750 50  0001 C CNN
 	1    6400 6750

Commit message: reorganize folder/files, added triple spacebar
Parts:
- added D_590, D_591: D, Diode_THT:D_DO-35_SOD27_P7.62mm_Horizontal, symbol Device:D_Small
- added K_610, K_612: KEYSW, MX_Only:MXOnly-2U-ReversedStabilizers-NoLED, symbol MX_Alps_Hybrid:MX-NoLED
- K_61: footprint MX_Only:MXOnly-6.25U-ReversedStabilizers-NoLED -> MX_Only:MXOnly-2.25U-ReversedStabilizers-NoLED
- SW1: symbol Env-KB60F-rescue:EVQ-P7A01P-PanasonicEVQ-P7A01P -> eec:EVQ-P7A01P
Connections:
- net col5: now also K_610.1 (COL)
- net col7: now also K_612.1 (COL)
- net row4: now also D_590.1 (K), D_591.1 (K)
- new net: D_590.2 (A), K_610.2 (ROW)
- new net: D_591.2 (A), K_612.2 (ROW)
Changed lines of the file:
@@
 F 0 "K_61" H 7400 5233 60  0000 C CNN
 F 1 "KEYSW" H 7400 4900 60  0001 C CNN
-F 2 "MX_Only:MXOnly-6.25U-ReversedStabilizers-NoLED" H 7400 5000 60  0001 C CNN
+F 2 "MX_Only:MXOnly-2.25U-ReversedStabilizers-NoLED" H 7400 5000 60  0001 C CNN
 F 3 "" H 7400 5000 60  0000 C CNN
 	1    7400 5000
@@
 	2350 5400 4350 5400
 Wire Wire Line
-	4350 5400 7350 5400
-Wire Wire Line
-	7350 5400 11350 5400
+	4350 5400 6350 5400
+Wire Wire Line
+	7350 5400 8350 5400
 Wire Wire Line
 	11350 5400 12350 5400
@@
 GND
 $Comp
-L Env-KB60F-rescue:EVQ-P7A01P-PanasonicEVQ-P7A01P SW1
+L eec:EVQ-P7A01P SW1
 U 1 1 6096F576
 P 3900 5950
@@
 Text GLabel 4200 7200 2    50   Input ~ 0
 VBUS
+$Comp
+L Device:D_Small D_590
+U 1 1 612E0015
+P 6350 5300
+F 0 "D_590" V 6420 5200 50  0000 R CNN
+F 1 "D" V 6330 5200 50  0000 R CNN
+F 2 "Diode_THT:D_DO-35_SOD27_P7.62mm_Horizontal" H 6050 5250 50  0001 C CNN
+F 3 "~" H 6050 5250 50  0001 C CNN
+	1    6350 5300
+	0    -1   -1   0
+$EndComp
+$Comp
+L Device:D_Small D_591
+U 1 1 612E0C96
+P 8350 5300
+F 0 "D_591" V 8420 5200 50  0000 R CNN
+F 1 "D" V 8330 5200 50  0000 R CNN
+F 2 "Diode_THT:D_DO-35_SOD27_P7.62mm_Horizontal" H 8050 5250 50  0001 C CNN
+F 3 "~" H 8050 5250 50  0001 C CNN
+	1    8350 5300
+	0    -1   -1   0
+$EndComp
+Connection ~ 8350 5400
+Wire Wire Line
+	8350 5400 11350 5400
+Connection ~ 6350 5400
+Wire Wire Line
+	6350 5400 7350 5400
+$Comp
+L MX_Alps_Hybrid:MX-NoLED K_610
+U 1 1 612E1979
+P 6400 5000
+F 0 "K_610" H 6400 5233 60  0000 C CNN
+F 1 "KEYSW" H 6400 4900 60  0001 C CNN
+F 2 "MX_Only:MXOnly-2U-ReversedStabilizers-NoLED" H 6400 5000 60  0001 C CNN
+F 3 "" H 6400 5000 60  0000 C CNN
+	1    6400 5000
+	1    0    0    -1
+$EndComp
+$Comp
+L MX_Alps_Hybrid:MX-NoLED K_612
+U 1 1 612E2128
+P 8400 5000
+F 0 "K_612" H 8400 5233 60  0000 C CNN
+F 1 "KEYSW" H 8400 4900 60  0001 C CNN
+F 2 "MX_Only:MXOnly-2U-ReversedStabilizers-NoLED" H 8400 5000 60  0001 C CNN
+F 3 "" H 8400 5000 60  0000 C CNN
+	1    8400 5000
+	1    0    0    -1
+$EndComp
+Wire Wire Line
+	6350 5200 6350 5150
+Wire Wire Line
+	8350 5200 8350 5150
+Wire Wire Line
+	6550 4950 6800 4950
+Wire Wire Line
+	6800 4950 6800 3950
+Connection ~ 6800 3950
+Wire Wire Line
+	8550 4950 8800 4950
+Wire Wire Line
+	8800 4950 8800 3950
+Connection ~ 8800 3950
 $EndSCHEMATC

Commit message: Corrected mount hole placement on all PCBs and updated the switch plate to fit triple spacebar split.
Parts:
- H1, H10, H11, H2, H3, H4, H5, H6, H7, H9: symbol Mechanical:MountingHole -> Mechanical:MountingHole_Pad
Connections:
- net GND: now also H1.1, H10.1, H11.1, H2.1, H3.1, H4.1, H5.1, H6.1, H7.1, H9.1
Changed lines of the file:
@@
-	1    0    0    -1
-$EndComp
-$Comp
-L Mechanical:MountingHole H1
-U 1 1 608AB119
-P 5600 6350
-F 0 "H1" H 5700 6396 50  0000 L CNN
-F 1 "MountingHole" H 5700 6305 50  0000 L CNN
-F 2 "AKLogo:MountingHole_2.2mm_M2-MODIFIED" H 5600 6350 50  0001 C CNN
-F 3 "~" H 5600 6350 50  0001 C CNN
-	1    5600 6350
-	1    0    0    -1
-$EndComp
-$Comp
-L Mechanical:MountingHole H3
-U 1 1 608ACB73
-P 5600 6550
-F 0 "H3" H 5700 6596 50  0000 L CNN
-F 1 "MountingHole" H 5700 6505 50  0000 L CNN
-F 2 "AKLogo:MountingHole_2.2mm_M2-MODIFIED" H 5600 6550 50  0001 C CNN
-F 3 "~" H 5600 6550 50  0001 C CNN
-	1    5600 6550
-	1    0    0    -1
-$EndComp
-$Comp
-L Mechanical:MountingHole H5
-U 1 1 608BCF9C
-P 5600 6750
-F 0 "H5" H 5700 6796 50  0000 L CNN
-F 1 "MountingHole" H 5700 6705 50  0000 L CNN
-F 2 "AKLogo:MountingHole_2.2mm_M2-MODIFIED" H 5600 6750 50  0001 C CNN
-F 3 "~" H 5600 6750 50  0001 C CNN
-	1    5600 6750
-	1    0    0    -1
-$EndComp
-$Comp
-L Mechanical:MountingHole H7
-U 1 1 608CD285
-P 5600 6950
-F 0 "H7" H 5700 6996 50  0000 L CNN
-F 1 "MountingHole" H 5700 6905 50  0000 L CNN
-F 2 "AKLogo:MountingHole_2.2mm_M2-MODIFIED" H 5600 6950 50  0001 C CNN
-F 3 "~" H 5600 6950 50  0001 C CNN
-	1    5600 6950
-	1    0    0    -1
-$EndComp
-$Comp
-L Mechanical:MountingHole H9
-U 1 1 608DD691
-P 5600 7150
-F 0 "H9" H 5700 7196 50  0000 L CNN
-F 1 "MountingHole" H 5700 7105 50  0000 L CNN
-F 2 "AKLogo:MountingHole_2.2mm_M2-MODIFIED" H 5600 7150 50  0001 C CNN
-F 3 "~" H 5600 7150 50  0001 C CNN
-	1    5600 7150
-	1    0    0    -1
-$EndComp
-$Comp
-L Mechanical:MountingHole H10
-U 1 1 608EDB63
-P 5600 7350
-F 0 "H10" H 5700 7396 50  0000 L CNN
-F 1 "MountingHole" H 5700 7305 50  0000 L CNN
-F 2 "AKLogo:MountingHole_2.2mm_M2-MODIFIED" H 5600 7350 50  0001 C CNN
-F 3 "~" H 5600 7350 50  0001 C CNN
-	1    5600 7350
-	1    0    0    -1
-$EndComp
-$Comp
-L Mechanical:MountingHole H11
-U 1 1 609431FD
-P 5600 7550
-F 0 "H11" H 5700 7596 50  0000 L CNN
-F 1 "MountingHole" H 5700 7505 50  0000 L CNN
-F 2 "AKLogo:MountingHole_2.2mm_M2-MODIFIED" H 5600 7550 50  0001 C CNN
-F 3 "~" H 5600 7550 50  0001 C CNN
-	1    5600 7550
 	1    0    0    -1
 $EndComp
@@
 Wire Wire Line
 	3950 5750 3950 5850
-$Comp
-L Mechanical:MountingHole H2
-U 1 1 609389EF
-P 6400 6350
-F 0 "H2" H 6500 6396 50  0000 L CNN
-F 1 "MountingHole" H 6500 6305 50  0000 L CNN
-F 2 "AKLogo:MountingHole_2.2mm_M2-MODIFIED" H 6400 6350 50  0001 C CNN
-F 3 "~" H 6400 6350 50  0001 C CNN
-	1    6400 6350
-	1    0    0    -1
-$EndComp
-$Comp
-L Mechanical:MountingHole H4
-U 1 1 609389F5
-P 6400 6550
-F 0 "H4" H 6500 6596 50  0000 L CNN
-F 1 "MountingHole" H 6500 6505 50  0000 L CNN
-F 2 "AKLogo:MountingHole_2.2mm_M2-MODIFIED" H 6400 6550 50  0001 C CNN
-F 3 "~" H 6400 6550 50  0001 C CNN
-	1    6400 6550
-	1    0    0    -1
-$EndComp
-$Comp
-L Mechanical:MountingHole H6
-U 1 1 609389FB
-P 6400 6750
-F 0 "H6" H 6500 6796 50  0000 L CNN
-F 1 "MountingHole" H 6500 6705 50  0000 L CNN
-F 2 "AKLogo:MountingHole_2.2mm_M2-MODIFIED" H 6400 6750 50  0001 C CNN
-F 3 "~" H 6400 6750 50  0001 C CNN
-	1    6400 6750
-	1    0    0    -1
-$EndComp
 $Comp
 L MX_Alps_Hybrid:MX-NoLED K_29
@@
 	8800 4950 8800 3950
 Connection ~ 8800 3950
+$Comp
+L Mechanical:MountingHole_Pad H6
+U 1 1 609389FB
+P 6400 6750
+F 0 "H6" H 6500 6796 50  0000 L CNN
+F 1 "MountingHole" H 6500 6705 50  0000 L CNN
+F 2 "AKLogo:MountingHole_2.2mm_M2-MODIFIED" H 6400 6750 50  0001 C CNN
+F 3 "~" H 6400 6750 50  0001 C CNN
+	1    6400 6750
+	0    -1   -1   0
+$EndComp
+$Comp
+L Mechanical:MountingHole_Pad H4
+U 1 1 609389F5
+P 6400 6550
+F 0 "H4" H 6500 6596 50  0000 L CNN
+F 1 "MountingHole" H 6500 6505 50  0000 L CNN
+F 2 "AKLogo:MountingHole_2.2mm_M2-MODIFIED" H 6400 6550 50  0001 C CNN
+F 3 "~" H 6400 6550 50  0001 C CNN
+	1    6400 6550
+	0    -1   -1   0
+$EndComp
+$Comp
+L Mechanical:MountingHole_Pad H2
+U 1 1 609389EF
+P 6400 6350
+F 0 "H2" H 6500 6396 50  0000 L CNN
+F 1 "MountingHole" H 6500 6305 50  0000 L CNN
+F 2 "AKLogo:MountingHole_2.2mm_M2-MODIFIED" H 6400 6350 50  0001 C CNN
+F 3 "~" H 6400 6350 50  0001 C CNN
+	1    6400 6350
+	0    -1   -1   0
+$EndComp
+$Comp
+L Mechanical:MountingHole_Pad H11
+U 1 1 609431FD
+P 6400 7750
+F 0 "H11" H 6500 7796 50  0000 L CNN
+F 1 "MountingHole" H 6500 7705 50  0000 L CNN
+F 2 "AKLogo:MountingHole_2.2mm_M2-MODIFIED" H 6400 7750 50  0001 C CNN
+F 3 "~" H 6400 7750 50  0001 C CNN
+	1    6400 7750
+	0    -1   -1   0
+$EndComp
+$Comp
+L Mechanical:MountingHole_Pad H10
+U 1 1 608EDB63
+P 6400 8150
+F 0 "H10" H 6500 8196 50  0000 L CNN
+F 1 "MountingHole" H 6500 8105 50  0000 L CNN
+F 2 "AKLogo:MountingHole_2.2mm_M2-MODIFIED" H 6400 8150 50  0001 C CNN
+F 3 "~" H 6400 8150 50  0001 C CNN
+	1    6400 8150
+	0    -1   -1   0
+$EndComp
+$Comp
+L Mechanical:MountingHole_Pad H9
+U 1 1 608DD691
+P 6400 7950
+F 0 "H9" H 6500 7996 50  0000 L CNN
+F 1 "MountingHole" H 6500 7905 50  0000 L CNN
+F 2 "AKLogo:MountingHole_2.2mm_M2-MODIFIED" H 6400 7950 50  0001 C CNN
+F 3 "~" H 6400 7950 50  0001 C CNN
+	1    6400 7950
+	0    -1   -1   0
+$EndComp
+$Comp
+L Mechanical:MountingHole_Pad H7
+U 1 1 608CD285
+P 6400 7550
+F 0 "H7" H 6500 7596 50  0000 L CNN
+F 1 "MountingHole" H 6500 7505 50  0000 L CNN
+F 2 "AKLogo:MountingHole_2.2mm_M2-MODIFIED" H 6400 7550 50  0001 C CNN
+F 3 "~" H 6400 7550 50  0001 C CNN
+	1    6400 7550
+	0    -1   -1   0
+$EndComp
+$Comp
+L Mechanical:MountingHole_Pad H5
+U 1 1 608BCF9C
+P 6400 7350
+F 0 "H5" H 6500 7396 50  0000 L CNN
+F 1 "MountingHole" H 6500 7305 50  0000 L CNN
+F 2 "AKLogo:MountingHole_2.2mm_M2-MODIFIED" H 6400 7350 50  0001 C CNN
+F 3 "~" H 6400 7350 50  0001 C CNN
+	1    6400 7350
+	0    -1   -1   0
+$EndComp
+$Comp
+L Mechanical:MountingHole_Pad H3
+U 1 1 608ACB73
+P 6400 7150
+F 0 "H3" H 6500 7196 50  0000 L CNN
+F 1 "MountingHole" H 6500 7105 50  0000 L CNN
+F 2 "AKLogo:MountingHole_2.2mm_M2-MODIFIED" H 6400 7150 50  0001 C CNN
+F 3 "~" H 6400 7150 50  0001 C CNN
+	1    6400 7150
+	0    -1   -1   0
+$EndComp
+$Comp
+L Mechanical:MountingHole_Pad H1
+U 1 1 608AB119
+P 6400 6950
+F 0 "H1" H 6500 6996 50  0000 L CNN
+F 1 "MountingHole" H 6500 6905 50  0000 L CNN
+F 2 "AKLogo:MountingHole_2.2mm_M2-MODIFIED" H 6400 6950 50  0001 C CNN
+F 3 "~" H 6400 6950 50  0001 C CNN
+	1    6400 6950
+	0    -1   -1   0
+$EndComp
+Wire Wire Line
+	6500 8150 6500 7950
+Wire Wire Line
+	6500 6350 6650 6350
+Connection ~ 6500 6350
+Connection ~ 6500 6550
+Wire Wire Line
+	6500 6550 6500 6350
+Connection ~ 6500 6750
+Wire Wire Line
+	6500 6750 6500 6550
+Connection ~ 6500 6950
+Wire Wire Line
+	6500 6950 6500 6750
+Connection ~ 6500 7150
+Wire Wire Line
+	6500 7150 6500 6950
+Connection ~ 6500 7350
+Wire Wire Line
+	6500 7350 6500 7150
+Connection ~ 6500 7550
+Wire Wire Line
+	6500 7550 6500 7350
+Connection ~ 6500 7750
+Wire Wire Line
+	6500 7750 6500 7550
+Connection ~ 6500 7950
+Wire Wire Line
+	6500 7950 6500 7750
+$Comp
+L power:GND #PWR?
+U 1 1 616E462A
+P 6650 6350
+F 0 "#PWR?" H 6650 6100 50  0001 C CNN
+F 1 "GND" V 6655 6222 50  0000 R CNN
+F 2 "" H 6650 6350 50  0001 C CNN
+F 3 "" H 6650 6350 50  0001 C CNN
+	1    6650 6350
+	0    -1   -1   0
+$EndComp
 $EndSCHEMATC
