File: MainPCB/Env-KB60F.kicad_sch (KiCad schematic)
At the start: 157 parts

Commit message: forgot to save schematic changes
Parts:
- USB1: footprint josh-connectors:USB_C_U262-161N-4BVC11 -> (none)
Changed lines of the file:
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@@
   (junction (at 34.29 111.76) (diameter 0) (color 0 0 0 0)
   )
-  (no_connect (at 39.37 186.69))
   (no_connect (at 39.37 189.23))
+  (no_connect (at 39.37 186.69))
   (wire (pts (xy 110.49 29.21) (xy 110.49 30.48))
     (stroke (width 0) (type default) (color 0 0 0 0))
@@
       (effects (font (size 1.524 1.524)))
     )
-    (property "Footprint" "josh-connectors:USB_C_U262-161N-4BVC11" (id 2) (at 24.13 173.99 0)
+    (property "Footprint" "" (id 2) (at 24.13 173.99 0)
       (effects (font (size 1.27 1.27)) hide)
     )
@@
     )
     (path "/00000000-0000-0000-0000-000060aaf05f"
-      (reference "5.1K1") (unit 1) (value "5.1K 0402 Resistor") (footprint "Resistor_SMD:R_0402_1005Metric")
+      (reference "5.1K1") (unit 1) (value "5.1K 0402 Resistor") (footprint "Resistor_THT:R_Axial_DIN0207_L6.3mm_D2.5mm_P10.16mm_Horizontal")
     )
     (path "/00000000-0000-0000-0000-000060aac80f"
-      (reference "5.1K2") (unit 1) (value "5.1K 0402 Resistor") (footprint "Resistor_SMD:R_0402_1005Metric")
+      (reference "5.1K2") (unit 1) (value "5.1K 0402 Resistor") (footprint "Resistor_THT:R_Axial_DIN0207_L6.3mm_D2.5mm_P10.16mm_Horizontal")
     )
     (path "/8512be71-fd68-4fcf-a580-ea27e3f43582"
@@
     )
     (path "/00000000-0000-0000-0000-000060a58fc0"
-      (reference "USB1") (unit 1) (value "HRO-TYPE-C-31-M-14") (footprint "josh-connectors:USB_C_U262-161N-4BVC11")
+      (reference "USB1") (unit 1) (value "HRO-TYPE-C-31-M-14") (footprint "josh-connectors:USB_C_TYPE-C-31-M-14")
     )
     (path "/6415485b-4a78-456e-b112-f1ce25139b4e"

Commit message: small tweaks regarding silkscreen
Parts:
- 5.1K1, 5.1K2: value (none) -> 5.1K 0402 Resistor; footprint (none) -> Resistor_THT:R_Axial_DIN0207_L6.3mm_D2.5mm_P10.16mm_Horizontal
- D_1, D_10, D_11, D_12, D_13, D_14, D_15, D_16, D_17, D_18, D_19, D_2, D_20, D_21, D_22, D_23, D_24, D_25, D_26, D_27, D_28, D_29, D_3, D_30, D_31, D_32, D_33, D_34, D_35, D_36, D_37, D_38, D_39, D_4, D_40, D_41, D_42, D_43, D_44, D_45, D_46, D_47, D_48, D_49, D_5, D_50, D_51, D_52, D_53, D_54, D_55, D_56, D_57, D_58, D_59, D_590, D_591, D_6, D_60, D_61, D_62, D_63, D_7, D_8, D_9: value (none) -> D; footprint (none) -> Diode_THT:D_DO-35_SOD27_P7.62mm_Horizontal
- H1, H10, H11, H2, H3, H4, H5, H6, H7, H9: value (none) -> MountingHole; footprint (none) -> Env_Extras:MountingHole_2.2mm_M2-MODIFIED
- J1: value (none) -> TP3 Pad; footprint (none) -> TestPoint:TestPoint_Pad_1.0x1.0mm
- J2: value (none) -> TP2 Pad; footprint (none) -> TestPoint:TestPoint_Pad_1.0x1.0mm
- K_1, K_10, K_11, K_12, K_13, K_14, K_15, K_16, K_17, K_18, K_19, K_2, K_20, K_21, K_22, K_23, K_24, K_25, K_26, K_27, K_28, K_29, K_3, K_30, K_31, K_32, K_33, K_34, K_35, K_36, K_37, K_38, K_39, K_4, K_40, K_41, K_42, K_43, K_44, K_45, K_46, K_47, K_48, K_49, K_5, K_50, K_51, K_52, K_53, K_54, K_55, K_56, K_57, K_58, K_59, K_6, K_60, K_61, K_610, K_612, K_62, K_63, K_64, K_65, K_7, K_8, K_9: value (none) -> KEYSW; footprint (none) -> MX_Only:MXOnly-1U-NoLED
- SW1: value (none) -> EVQ-P7A01P; footprint (none) -> PanasonicEVQ-P7A01P:Panasonic-EVQ-P7A01P-0-0-MFG
- U1: value (none) -> Pico; footprint (none) -> MCU_RaspberryPi_and_Boards:RPi_Pico_SMD_TH
- USB1: value (none) -> HRO-TYPE-C-31-M-14; footprint (none) -> josh-connectors:USB_C_TYPE-C-31-M-14
- stab1, stab2, stab3, stab4, stab5, stab6, stab7, stab8: value (none) -> MX Stabilizer; footprint (none) -> Mounting_Keyboard_Stabilizer:Stabilizer_Cherry_MX_2u
