File: MainPCB-HS/Env-KB60FHS.kicad_pcb (KiCad board)
At the start: 2 copper layers, 283 x 126.5 mm, 149 parts, among them J1 TP3 Pad, J2 TP2 Pad, SW1 EVQ-P7A01P, U1 Pico

Commit message: finished up hotswap version traces
Routing:
- net Net-(D_62-Pad2): track 6.05 -> 171.7 mm
- net Net-(D_61-Pad2): track 5.49 -> 168.5 mm
- net Net-(D_60-Pad2): track 6.34 -> 164.5 mm
- net Net-(D_55-Pad2): track 5.42 -> 157.9 mm
- net Net-(D_54-Pad2): track 4.78 -> 144.4 mm
- net Net-(D_53-Pad2): track 5.70 -> 143.4 mm
- net Net-(D_63-Pad2): track 19.9 -> 155.5 mm
- net Net-(D_41-Pad2): track 4.78 -> 127.3 mm
- net Net-(D_42-Pad2): track 15.4 -> 136.0 mm, vias 0 -> 1
- net Net-(D_40-Pad2): track 5.77 -> 122.3 mm
- net Net-(D_39-Pad2): track 4.07 -> 115.1 mm
- net Net-(D_38-Pad2): track 5.06 -> 111.4 mm
- net Net-(D_28-Pad2): track 9.93 -> 92.3 mm
- net Net-(D_26-Pad2): track 5.13 -> 80.7 mm
- net Net-(D_27-Pad2): track 11.1 -> 86.2 mm
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