File: BackPCB/EnvKB60F-BackPlate.kicad_pcb (KiCad board)
At the start: 2 copper layers, 283 x 126.5 mm, 9 parts

Commit message: updated backplate
Parts:
- added kibuzzard-627532E1: G***, kibuzzard-627532E1, F.Cu at (91.5, 44.5)
Other:
- net class Default removed
- net class USB removed
