File: SwitchPlate/EnvKB60F-SwitchPlate.kicad_pcb (KiCad board)
At the start: 2 copper layers, 283 x 126.5 mm, 0 parts

Commit message: Re-created switchplate
Parts:
- added H1: MountingHole, Env_Extras:MountingHole_2.2mm_M2_DIN965_Pad-MODIFIED, F.Cu at (227.5, 155.0)
- added H10: MountingHole, Env_Extras:MountingHole_2.2mm_M2_DIN965_Pad-MODIFIED, F.Cu at (314.1, 84.1)
- added H11: MountingHole, Env_Extras:MountingHole_2.2mm_M2_DIN965_Pad-MODIFIED, F.Cu at (353.1, 36.5)
- added H2: MountingHole, Env_Extras:MountingHole_2.2mm_M2_DIN965_Pad-MODIFIED, F.Cu at (99.8, 155.5)
- added H3: MountingHole, Env_Extras:MountingHole_2.2mm_M2_DIN965_Pad-MODIFIED, F.Cu at (87.0, 38.1)
- added H4: MountingHole, Env_Extras:MountingHole_2.2mm_M2_DIN965_Pad-MODIFIED, F.Cu at (101.8, 84.1)
- added H6: MountingHole, Env_Extras:MountingHole_2.2mm_M2_DIN965_Pad-MODIFIED, F.Cu at (338.0, 155.5)
- added H9: MountingHole, Env_Extras:MountingHole_2.2mm_M2_DIN965_Pad-MODIFIED, F.Cu at (218.5, 84.0)
- added K_1: KEYSW, Env_Extras:MXOnly-1U-Mask, F.Cu at (85.5, 74.5)
- added K_10: KEYSW, Env_Extras:MXOnly-1U-Mask, F.Cu at (257.0, 74.5)
- added K_11: KEYSW, Env_Extras:MXOnly-1U-Mask, F.Cu at (276.0, 74.5)
- added K_12: KEYSW, Env_Extras:MXOnly-1U-Mask, F.Cu at (295.1, 74.5)
- added K_13: KEYSW, Env_Extras:MXOnly-1U-Mask, F.Cu at (314.1, 74.5)
- added K_14: KEYSW, Env_Extras:MXOnly-1U-Mask, F.Cu at (342.7, 74.5)
- added K_15: KEYSW, Env_Extras:MXOnly-1U-Mask, F.Cu at (90.3, 93.6)
- added K_16: KEYSW, Env_Extras:MXOnly-1U-Mask, F.Cu at (114.1, 93.6)
- added K_17: KEYSW, Env_Extras:MXOnly-1U-Mask, F.Cu at (133.2, 93.6)
- added K_18: KEYSW, Env_Extras:MXOnly-1U-Mask, F.Cu at (152.2, 93.6)
- added K_19: KEYSW, Env_Extras:MXOnly-1U-Mask, F.Cu at (171.2, 93.6)
- added K_2: KEYSW, Env_Extras:MXOnly-1U-Mask, F.Cu at (104.6, 74.5)
- added K_20: KEYSW, Env_Extras:MXOnly-1U-Mask, F.Cu at (190.3, 93.6)
- added K_21: KEYSW, Env_Extras:MXOnly-1U-Mask, F.Cu at (209.3, 93.6)
- added K_22: KEYSW, Env_Extras:MXOnly-1U-Mask, F.Cu at (228.4, 93.6)
- added K_23: KEYSW, Env_Extras:MXOnly-1U-Mask, F.Cu at (247.4, 93.6)
- added K_24: KEYSW, Env_Extras:MXOnly-1U-Mask, F.Cu at (266.5, 93.6)
- added K_25: KEYSW, Env_Extras:MXOnly-1U-Mask, F.Cu at (285.6, 93.6)
- added K_26: KEYSW, Env_Extras:MXOnly-1U-Mask, F.Cu at (304.6, 93.6)
- added K_27: KEYSW, Env_Extras:MXOnly-1U-Mask, F.Cu at (323.6, 93.6)
- added K_28: KEYSW, Env_Extras:MXOnly-1U-Mask, F.Cu at (347.4, 93.5)
- added K_29: KEYSW, Env_Extras:MXOnly-1U-Mask, F.Cu at (340.3, 112.6)
- added K_3: KEYSW, Env_Extras:MXOnly-1U-Mask, F.Cu at (123.6, 74.5)
- added K_30: KEYSW, Env_Extras:MXOnly-1U-Mask, F.Cu at (92.7, 112.6)
- added K_31: KEYSW, Env_Extras:MXOnly-1U-Mask, F.Cu at (118.9, 112.6)
- added K_32: KEYSW, Env_Extras:MXOnly-1U-Mask, F.Cu at (137.9, 112.6)
- added K_33: KEYSW, Env_Extras:MXOnly-1U-Mask, F.Cu at (157.0, 112.6)
- added K_34: KEYSW, Env_Extras:MXOnly-1U-Mask, F.Cu at (176.0, 112.6)
- added K_35: KEYSW, Env_Extras:MXOnly-1U-Mask, F.Cu at (195.1, 112.6)
- added K_36: KEYSW, Env_Extras:MXOnly-1U-Mask, F.Cu at (214.1, 112.6)
- added K_37: KEYSW, Env_Extras:MXOnly-1U-Mask, F.Cu at (233.2, 112.6)
- added K_38: KEYSW, Env_Extras:MXOnly-1U-Mask, F.Cu at (252.2, 112.6)
- added K_39: KEYSW, Env_Extras:MXOnly-1U-Mask, F.Cu at (271.3, 112.6)
- added K_4: KEYSW, Env_Extras:MXOnly-1U-Mask, F.Cu at (142.7, 74.5)
- added K_40: KEYSW, Env_Extras:MXOnly-1U-Mask, F.Cu at (290.3, 112.6)
- added K_41: KEYSW, Env_Extras:MXOnly-1U-Mask, F.Cu at (309.4, 112.6)
- added K_42: KEYSW, Env_Extras:MXOnly-1U-Mask, F.Cu at (328.4, 112.6)
- added K_43: KEYSW, Env_Extras:MXOnly-1U-Mask, F.Cu at (349.8, 103.1)
- added K_44: KEYSW, Env_Extras:MXOnly-1U-Mask, F.Cu at (97.4, 131.7)
- added K_45: KEYSW, Env_Extras:MXOnly-1U-Mask, F.Cu at (87.9, 131.7)
- added K_46: KEYSW, Env_Extras:MXOnly-1U-Mask, F.Cu at (109.3, 131.7)
- added K_47: KEYSW, Env_Extras:MXOnly-1U-Mask, F.Cu at (128.4, 131.7)
- added K_48: KEYSW, Env_Extras:MXOnly-1U-Mask, F.Cu at (147.4, 131.7)
- added K_49: KEYSW, Env_Extras:MXOnly-1U-Mask, F.Cu at (166.5, 131.7)
- added K_5: KEYSW, Env_Extras:MXOnly-1U-Mask, F.Cu at (161.7, 74.5)
- added K_50: KEYSW, Env_Extras:MXOnly-1U-Mask, F.Cu at (185.5, 131.7)
- added K_51: KEYSW, Env_Extras:MXOnly-1U-Mask, F.Cu at (204.6, 131.7)
- added K_52: KEYSW, Env_Extras:MXOnly-1U-Mask, F.Cu at (223.6, 131.7)
- added K_53: KEYSW, Env_Extras:MXOnly-1U-Mask, F.Cu at (242.7, 131.7)
- added K_54: KEYSW, Env_Extras:MXOnly-1U-Mask, F.Cu at (261.7, 131.7)
- added K_55: KEYSW, Env_Extras:MXOnly-1U-Mask, F.Cu at (280.8, 131.7)
- added K_56: KEYSW, Env_Extras:MXOnly-1U-Mask, F.Cu at (299.8, 131.7)
- added K_57: KEYSW, Env_Extras:MXOnly-1U-Mask, F.Cu at (335.6, 131.7)
- added K_58: KEYSW, Env_Extras:MXOnly-1U-Mask, F.Cu at (87.9, 150.7)
- added K_59: KEYSW, Env_Extras:MXOnly-1U-Mask, F.Cu at (111.7, 150.7)
- added K_6: KEYSW, Env_Extras:MXOnly-1U-Mask, F.Cu at (180.8, 74.5)
- added K_60: KEYSW, Env_Extras:MXOnly-1U-Mask, F.Cu at (135.5, 150.7)
- added K_61: KEYSW, Env_Extras:MXOnly-1U-Mask, F.Cu at (207.0, 150.7)
- added K_610: KEYSW, Env_Extras:MXOnly-1U-Mask, F.Cu at (166.5, 150.7)
- added K_612: KEYSW, Env_Extras:MXOnly-1U-Mask, F.Cu at (247.4, 150.7)
- added K_62: KEYSW, Env_Extras:MXOnly-1U-Mask, F.Cu at (278.4, 150.7)
- added K_63: KEYSW, Env_Extras:MXOnly-1U-Mask, F.Cu at (302.2, 150.7)
- added K_64: KEYSW, Env_Extras:MXOnly-1U-Mask, F.Cu at (326.0, 150.7)
- added K_65: KEYSW, Env_Extras:MXOnly-1U-Mask, F.Cu at (349.8, 150.7)
- added K_7: KEYSW, Env_Extras:MXOnly-1U-Mask, F.Cu at (199.8, 74.5)
- added K_8: KEYSW, Env_Extras:MXOnly-1U-Mask, F.Cu at (218.9, 74.5)
- added K_9: KEYSW, Env_Extras:MXOnly-1U-Mask, F.Cu at (237.9, 74.5)
Routing:
- added copper zone on B.Cu, net GND
- added copper zone on F.Cu, net GND
- removed copper zone on B.Cu, net (none)
- removed copper zone on F.Cu, net (none)
Other:
- outline, holes or cut-outs redrawn
- net class Default removed
- net class USB removed
- board text added: "RESET MCU"
- board text removed: "Envious.Media"

Commit message: updated switch plate
Other:
- outline, holes or cut-outs redrawn
- board text removed: "RESET MCU"
