File: MainPCB_ChocV2/Env-KB60C2.kicad_sch (KiCad schematic)
At the start: 157 parts, among them J1 TP3 Pad, J2 TP2 Pad, SW1 EVQ-P7A01P, U1 Pico

Commit message: some various corrections to the USB DP/DM traces
Parts:
- U1: footprint MCU_RaspberryPi_and_Boards:RPi_Pico_SMD_TH -> MCU_RaspberryPi_and_Boards:RPi_Pico_SMD_TH_MODIFIED
Changed lines of the file:
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@@
     (property "Reference" "U1" (id 0) (at 102.87 177.8 0))
     (property "Value" "Pico" (id 1) (at 99.06 177.8 0))
-    (property "Footprint" "MCU_RaspberryPi_and_Boards:RPi_Pico_SMD_TH" (id 2) (at 88.9 207.01 90)
+    (property "Footprint" "MCU_RaspberryPi_and_Boards:RPi_Pico_SMD_TH_MODIFIED" (id 2) (at 88.9 207.01 90)
       (effects (font (size 1.27 1.27)) hide)
     )
@@
     )
     (path "/00000000-0000-0000-0000-00006095eae7"
-      (reference "U1") (unit 1) (value "Pico") (footprint "MCU_RaspberryPi_and_Boards:RPi_Pico_SMD_TH")
+      (reference "U1") (unit 1) (value "Pico") (footprint "MCU_RaspberryPi_and_Boards:RPi_Pico_SMD_TH_MODIFIED")
     )
     (path "/00000000-0000-0000-0000-000060a58fc0"

Commit message: swapped mount holes
Parts:
- H1, H10, H11, H2, H3, H4, H5, H6, H7, H9: footprint Env_Extras:MountingHole_2.2mm_M2-MODIFIED -> Env_Extras:MountingHole_2.2mm_M2_DIN965_Pad-MODIFIED
Changed lines of the file:
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@@
       (effects (font (size 1.27 1.27)) (justify left))
     )
-    (property "Footprint" "Env_Extras:MountingHole_2.2mm_M2-MODIFIED" (id 2) (at 162.56 176.53 0)
+    (property "Footprint" "Env_Extras:MountingHole_2.2mm_M2_DIN965_Pad-MODIFIED" (id 2) (at 162.56 176.53 0)
       (effects (font (size 1.27 1.27)) hide)
     )
@@
       (effects (font (size 1.27 1.27)) (justify left))
     )
-    (property "Footprint" "Env_Extras:MountingHole_2.2mm_M2-MODIFIED" (id 2) (at 162.56 181.61 0)
+    (property "Footprint" "Env_Extras:MountingHole_2.2mm_M2_DIN965_Pad-MODIFIED" (id 2) (at 162.56 181.61 0)
       (effects (font (size 1.27 1.27)) hide)
     )
@@
       (effects (font (size 1.27 1.27)) (justify left))
     )
-    (property "Footprint" "Env_Extras:MountingHole_2.2mm_M2-MODIFIED" (id 2) (at 162.56 186.69 0)
+    (property "Footprint" "Env_Extras:MountingHole_2.2mm_M2_DIN965_Pad-MODIFIED" (id 2) (at 162.56 186.69 0)
       (effects (font (size 1.27 1.27)) hide)
     )
@@
       (effects (font (size 1.27 1.27)) (justify left))
     )
-    (property "Footprint" "Env_Extras:MountingHole_2.2mm_M2-MODIFIED" (id 2) (at 162.56 191.77 0)
+    (property "Footprint" "Env_Extras:MountingHole_2.2mm_M2_DIN965_Pad-MODIFIED" (id 2) (at 162.56 191.77 0)
       (effects (font (size 1.27 1.27)) hide)
     )
@@
       (effects (font (size 1.27 1.27)) (justify left))
     )
-    (property "Footprint" "Env_Extras:MountingHole_2.2mm_M2-MODIFIED" (id 2) (at 162.56 201.93 0)
+    (property "Footprint" "Env_Extras:MountingHole_2.2mm_M2_DIN965_Pad-MODIFIED" (id 2) (at 162.56 201.93 0)
       (effects (font (size 1.27 1.27)) hide)
     )
@@
       (effects (font (size 1.27 1.27)) (justify left))
     )
-    (property "Footprint" "Env_Extras:MountingHole_2.2mm_M2-MODIFIED" (id 2) (at 162.56 207.01 0)
+    (property "Footprint" "Env_Extras:MountingHole_2.2mm_M2_DIN965_Pad-MODIFIED" (id 2) (at 162.56 207.01 0)
       (effects (font (size 1.27 1.27)) hide)
     )
@@
       (effects (font (size 1.27 1.27)) (justify left))
     )
-    (property "Footprint" "Env_Extras:MountingHole_2.2mm_M2-MODIFIED" (id 2) (at 162.56 161.29 0)
+    (property "Footprint" "Env_Extras:MountingHole_2.2mm_M2_DIN965_Pad-MODIFIED" (id 2) (at 162.56 161.29 0)
       (effects (font (size 1.27 1.27)) hide)
     )
@@
       (effects (font (size 1.27 1.27)) (justify left))
     )
-    (property "Footprint" "Env_Extras:MountingHole_2.2mm_M2-MODIFIED" (id 2) (at 162.56 166.37 0)
+    (property "Footprint" "Env_Extras:MountingHole_2.2mm_M2_DIN965_Pad-MODIFIED" (id 2) (at 162.56 166.37 0)
       (effects (font (size 1.27 1.27)) hide)
     )
@@
       (effects (font (size 1.27 1.27)) (justify left))
     )
-    (property "Footprint" "Env_Extras:MountingHole_2.2mm_M2-MODIFIED" (id 2) (at 162.56 171.45 0)
+    (property "Footprint" "Env_Extras:MountingHole_2.2mm_M2_DIN965_Pad-MODIFIED" (id 2) (at 162.56 171.45 0)
       (effects (font (size 1.27 1.27)) hide)
     )
@@
       (effects (font (size 1.27 1.27)) (justify left))
     )
-    (property "Footprint" "Env_Extras:MountingHole_2.2mm_M2-MODIFIED" (id 2) (at 162.56 196.85 0)
+    (property "Footprint" "Env_Extras:MountingHole_2.2mm_M2_DIN965_Pad-MODIFIED" (id 2) (at 162.56 196.85 0)
       (effects (font (size 1.27 1.27)) hide)
     )
@@
     )
     (path "/00000000-0000-0000-0000-0000608ab119"
-      (reference "H1") (unit 1) (value "MountingHole") (footprint "Env_Extras:MountingHole_2.2mm_M2-MODIFIED")
+      (reference "H1") (unit 1) (value "MountingHole") (footprint "Env_Extras:MountingHole_2.2mm_M2_DIN965_Pad-MODIFIED")
     )
     (path "/00000000-0000-0000-0000-0000609389ef"
-      (reference "H2") (unit 1) (value "MountingHole") (footprint "Env_Extras:MountingHole_2.2mm_M2-MODIFIED")
+      (reference "H2") (unit 1) (value "MountingHole") (footprint "Env_Extras:MountingHole_2.2mm_M2_DIN965_Pad-MODIFIED")
     )
     (path "/00000000-0000-0000-0000-0000608acb73"
-      (reference "H3") (unit 1) (value "MountingHole") (footprint "Env_Extras:MountingHole_2.2mm_M2-MODIFIED")
+      (reference "H3") (unit 1) (value "MountingHole") (footprint "Env_Extras:MountingHole_2.2mm_M2_DIN965_Pad-MODIFIED")
     )
     (path "/00000000-0000-0000-0000-0000609389f5"
-      (reference "H4") (unit 1) (value "MountingHole") (footprint "Env_Extras:MountingHole_2.2mm_M2-MODIFIED")
+      (reference "H4") (unit 1) (value "MountingHole") (footprint "Env_Extras:MountingHole_2.2mm_M2_DIN965_Pad-MODIFIED")
     )
     (path "/00000000-0000-0000-0000-0000608bcf9c"
-      (reference "H5") (unit 1) (value "MountingHole") (footprint "Env_Extras:MountingHole_2.2mm_M2-MODIFIED")
+      (reference "H5") (unit 1) (value "MountingHole") (footprint "Env_Extras:MountingHole_2.2mm_M2_DIN965_Pad-MODIFIED")
     )
     (path "/00000000-0000-0000-0000-0000609389fb"
-      (reference "H6") (unit 1) (value "MountingHole") (footprint "Env_Extras:MountingHole_2.2mm_M2-MODIFIED")
+      (reference "H6") (unit 1) (value "MountingHole") (footprint "Env_Extras:MountingHole_2.2mm_M2_DIN965_Pad-MODIFIED")
     )
     (path "/00000000-0000-0000-0000-0000608cd285"
-      (reference "H7") (unit 1) (value "MountingHole") (footprint "Env_Extras:MountingHole_2.2mm_M2-MODIFIED")
+      (reference "H7") (unit 1) (value "MountingHole") (footprint "Env_Extras:MountingHole_2.2mm_M2_DIN965_Pad-MODIFIED")
     )
     (path "/00000000-0000-0000-0000-0000608dd691"
-      (reference "H9") (unit 1) (value "MountingHole") (footprint "Env_Extras:MountingHole_2.2mm_M2-MODIFIED")
+      (reference "H9") (unit 1) (value "MountingHole") (footprint "Env_Extras:MountingHole_2.2mm_M2_DIN965_Pad-MODIFIED")
     )
     (path "/00000000-0000-0000-0000-0000608edb63"
-      (reference "H10") (unit 1) (value "MountingHole") (footprint "Env_Extras:MountingHole_2.2mm_M2-MODIFIED")
+      (reference "H10") (unit 1) (value "MountingHole") (footprint "Env_Extras:MountingHole_2.2mm_M2_DIN965_Pad-MODIFIED")
     )
     (path "/00000000-0000-0000-0000-0000609431fd"
-      (reference "H11") (unit 1) (value "MountingHole") (footprint "Env_Extras:MountingHole_2.2mm_M2-MODIFIED")
+      (reference "H11") (unit 1) (value "MountingHole") (footprint "Env_Extras:MountingHole_2.2mm_M2_DIN965_Pad-MODIFIED")
     )
     (path "/00000000-0000-0000-0000-000060b4329c"
