File: KiCad Files/BackPCB/60FBackplate.kicad_pcb (KiCad board)
At the start: 2 copper layers, 283 x 126.5 mm, 9 parts

Commit message: Decided extended plates are the norm.
Parts:
- removed H1, H10, H11, H2, H3, H4, H6, H9: MountingHole, Env_Extras:MountingHole_2.2mm_M2-MODIFIED
Other:
- board size 283 x 126.5 mm -> 287 x 132.5 mm
